File: thingTouch-Buttons/v1.0/_saved_thingTouch-Buttons_v1P0.sch (KiCad schematic (older format))
At the start: 23 parts, among them P1 DIRECT_CONN, P2 TOUCH_CONN, U1 TTP224N-BSB

Commit message: final routing done; verification left
Changed lines of the file:
@@
 F 0 "P1" H 2275 2025 50  0000 C CNN
 F 1 "DIRECT_CONN" V 2375 1675 50  0000 C CNN
-F 2 "Connectors_JST:JST_PH_S6B-PH-SM4-TB_06x2.00mm_Angled" H 2275 1675 50  0000 C CNN
+F 2 "Connectors_JST:JST_PH_S6B-PH-SM4-TB_06x2.00mm_Angled" H 2300 2125 50  0001 C CNN
 F 3 "" H 2275 1675 50  0000 C CNN
 	1    2275 1675
