File: thingTouch-Buttons/v1.0/thingTouch-Buttons_v1P0.sch (KiCad schematic (older format))
At the start: 23 parts, among them P1 DIRECT_CONN, P2 TOUCH_CONN, U1 TTP224N-BSB

Commit message: basic routing done
Parts:
- C1, C2, C3, C4, C5: footprint (none) -> Capacitors_SMD:C_0805_HandSoldering
- D1, D2, D3: footprint (none) -> LEDs:LED_0805_HandSoldering
- P1: footprint (none) -> Connectors_JST:JST_PH_S4B-PH-SM4-TB_04x2.00mm_Angled
- P2: footprint (none) -> Connectors_JST:JST_PH_S5B-PH-SM4-TB_05x2.00mm_Angled
- R1, R2, R3, R4, R5, R6, R7, R8, R9: footprint (none) -> Resistors_SMD:R_0805_HandSoldering
- U1: footprint (none) -> Housings_SSOP:SSOP-16_3.9x4.9mm_Pitch0.635mm
- W1, W2, W3: footprint (none) -> conn-wire-pads:TouchPad-round-1000
Connections:
- wire segments 70 -> 71
Changed lines of the file:
@@
 F 0 "W1" H 975 2650 60  0000 C CNN
 F 1 "touchPad" H 975 2250 60  0000 C CNN
-F 2 "" H 975 2450 60  0001 C CNN
+F 2 "conn-wire-pads:TouchPad-round-1000" H 975 2450 60  0001 C CNN
 F 3 "" H 975 2450 60  0001 C CNN
 	1    975  2450
@@
 F 0 "W2" H 975 3250 60  0000 C CNN
 F 1 "touchPad" H 975 2850 60  0000 C CNN
-F 2 "" H 975 3050 60  0001 C CNN
+F 2 "conn-wire-pads:TouchPad-round-1000" H 975 3050 60  0001 C CNN
 F 3 "" H 975 3050 60  0001 C CNN
 	1    975  3050
@@
 F 0 "W3" H 975 3925 60  0000 C CNN
 F 1 "touchPad" H 975 3525 60  0000 C CNN
-F 2 "" H 975 3725 60  0001 C CNN
+F 2 "conn-wire-pads:TouchPad-round-1000" H 975 3725 60  0001 C CNN
 F 3 "" H 975 3725 60  0001 C CNN
 	1    975  3725
@@
 F 0 "C1" H 1885 2645 50  0000 L CNN
 F 1 "30pF" H 1885 2495 50  0000 L CNN
-F 2 "" H 1875 2575 50  0000 C CNN
+F 2 "Capacitors_SMD:C_0805_HandSoldering" H 1875 2575 50  0001 C CNN
 F 3 "" H 1875 2575 50  0000 C CNN
 	1    1875 2575
@@
 F 0 "C2" H 1885 3245 50  0000 L CNN
 F 1 "30pF" H 1885 3095 50  0000 L CNN
-F 2 "" H 1875 3175 50  0000 C CNN
+F 2 "Capacitors_SMD:C_0805_HandSoldering" H 1875 3175 50  0001 C CNN
 F 3 "" H 1875 3175 50  0000 C CNN
 	1    1875 3175
@@
 F 0 "C3" H 1885 3920 50  0000 L CNN
 F 1 "30pF" H 1885 3770 50  0000 L CNN
-F 2 "" H 1875 3850 50  0000 C CNN
+F 2 "Capacitors_SMD:C_0805_HandSoldering" H 1875 3850 50  0001 C CNN
 F 3 "" H 1875 3850 50  0000 C CNN
 	1    1875 3850
@@
 F 0 "U1" H 3975 4350 60  0000 C CNN
 F 1 "TTP224N-BSB" H 3975 4200 60  0000 C CNN
-F 2 "" H 3975 4350 60  0001 C CNN
+F 2 "Housings_SSOP:SSOP-16_3.9x4.9mm_Pitch0.635mm" H 3975 4350 60  0001 C CNN
 F 3 "" H 3975 4350 60  0001 C CNN
 	1    3975 4350
@@
 L CONN_01X04 P1
 U 1 1 596D0BC9
-P 2275 1775
-F 0 "P1" H 2275 2025 50  0000 C CNN
-F 1 "DIRECT_CONN" V 2375 1775 50  0000 C CNN
-F 2 "" H 2275 1775 50  0000 C CNN
-F 3 "" H 2275 1775 50  0000 C CNN
-	1    2275 1775
+P 2275 1675
+F 0 "P1" H 2275 1925 50  0000 C CNN
+F 1 "DIRECT_CONN" V 2375 1675 50  0000 C CNN
+F 2 "Connectors_JST:JST_PH_S4B-PH-SM4-TB_04x2.00mm_Angled" H 2275 1675 50  0001 C CNN
+F 3 "" H 2275 1675 50  0000 C CNN
+	1    2275 1675
 	1    0    0    -1
 $EndComp
@@
 Wire Wire Line
 	2075 1825 1550 1825
-Wire Wire Line
-	1550 1825 1550 3725
 Connection ~ 1550 3725
 Wire Wire Line
 	1475 1725 2075 1725
 Connection ~ 1475 3050
-Wire Wire Line
-	1475 3050 1475 1725
-Wire Wire Line
-	1400 1625 1400 2450
-Connection ~ 1400 2450
 $Comp
 L GND #PWR02
 U 1 1 596D1262
-P 1950 1975
-F 0 "#PWR02" H 1950 2025 30  0001 C CNN
-F 1 "GND" H 1950 1850 30  0001 C CNN
-F 2 "" H 1950 1975 60  0000 C CNN
-F 3 "" H 1950 1975 60  0000 C CNN
-	1    1950 1975
-	1    0    0    -1
-$EndComp
-Wire Wire Line
-	2075 1925 1950 1925
-Wire Wire Line
-	1950 1925 1950 1975
+P 1825 1475
+F 0 "#PWR02" H 1825 1525 30  0001 C CNN
+F 1 "GND" H 1825 1350 30  0001 C CNN
+F 2 "" H 1825 1475 60  0000 C CNN
+F 3 "" H 1825 1475 60  0000 C CNN
+	1    1825 1475
+	1    0    0    -1
+$EndComp
+Wire Wire Line
+	1825 1425 2075 1425
+Wire Wire Line
+	1825 1425 1825 1475
 $Comp
 L VDD #PWR03
@@
 F 0 "R1" V 2925 4375 50  0000 L CNN
 F 1 "0E" V 3000 4350 50  0000 L CNN
-F 2 "" H 3000 4400 50  0000 C CNN
+F 2 "Resistors_SMD:R_0805_HandSoldering" H 3000 4400 50  0001 C CNN
 F 3 "" H 3000 4400 50  0000 C CNN
 	1    3000 4400
@@
 F 0 "R2" V 2950 4675 50  0000 L CNN
 F 1 "0E" V 3000 4550 50  0000 L CNN
-F 2 "" H 3000 4600 50  0000 C CNN
+F 2 "Resistors_SMD:R_0805_HandSoldering" H 3000 4600 50  0001 C CNN
 F 3 "" H 3000 4600 50  0000 C CNN
 	1    3000 4600
@@
 F 0 "R3" V 3050 4775 50  0000 L CNN
 F 1 "0E" V 3000 4650 50  0000 L CNN
-F 2 "" H 3000 4700 50  0000 C CNN
+F 2 "Resistors_SMD:R_0805_HandSoldering" H 3000 4700 50  0001 C CNN
 F 3 "" H 3000 4700 50  0000 C CNN
 	1    3000 4700
@@
 F 0 "C5" H 2600 4800 50  0000 L CNN
 F 1 "10uF" H 2600 4600 50  0000 L CNN
-F 2 "" H 2613 4550 50  0000 C CNN
+F 2 "Capacitors_SMD:C_0805_HandSoldering" H 2613 4550 50  0001 C CNN
 F 3 "" H 2575 4700 50  0000 C CNN
 	1    2575 4700
@@
 F 0 "C4" H 2325 4800 50  0000 L CNN
 F 1 "100nF" H 2025 4600 50  0000 L CNN
-F 2 "" H 2338 4550 50  0000 C CNN
+F 2 "Capacitors_SMD:C_0805_HandSoldering" H 2338 4550 50  0001 C CNN
 F 3 "" H 2300 4700 50  0000 C CNN
 	1    2300 4700
@@
 F 0 "R5" V 5125 4575 50  0000 L CNN
 F 1 "0E" V 5075 4450 50  0000 L CNN
-F 2 "" H 5075 4500 50  0000 C CNN
+F 2 "Resistors_SMD:R_0805_HandSoldering" H 5075 4500 50  0001 C CNN
 F 3 "" H 5075 4500 50  0000 C CNN
 	1    5075 4500
@@
 F 0 "R6" V 5125 4775 50  0000 L CNN
 F 1 "0E" V 5075 4650 50  0000 L CNN
-F 2 "" H 5075 4700 50  0000 C CNN
+F 2 "Resistors_SMD:R_0805_HandSoldering" H 5075 4700 50  0001 C CNN
 F 3 "" H 5075 4700 50  0000 C CNN
 	1    5075 4700
@@
 F 0 "R4" V 5125 4475 50  0000 L CNN
 F 1 "0E" V 5075 4350 50  0000 L CNN
-F 2 "" H 5075 4400 50  0000 C CNN
+F 2 "Resistors_SMD:R_0805_HandSoldering" H 5075 4400 50  0001 C CNN
 F 3 "" H 5075 4400 50  0000 C CNN
 	1    5075 4400
@@
 	4825 4000 5350 4000
 Wire Wire Line
-	4925 4000 4925 3175
-Wire Wire Line
 	4925 3175 5225 3175
 Wire Wire Line
@@
 	4825 4200 5125 4200
 Wire Wire Line
-	5125 3375 5125 4300
-Wire Wire Line
 	5125 3375 5225 3375
-Wire Wire Line
-	5025 4100 5025 3275
 Wire Wire Line
 	5025 3275 5225 3275
@@
 F 0 "P2" H 5425 3475 50  0000 C CNN
 F 1 "TOUCH_CONN" V 5525 3175 50  0000 C CNN
-F 2 "" H 5425 3175 50  0000 C CNN
+F 2 "Connectors_JST:JST_PH_S5B-PH-SM4-TB_05x2.00mm_Angled" H 5425 3175 50  0001 C CNN
 F 3 "" H 5425 3175 50  0000 C CNN
 	1    5425 3175
@@
 F 0 "D2" H 5675 4125 50  0000 L CNN
 F 1 "LED1" H 5800 3950 50  0000 L CNN
-F 2 "" V 5725 4000 50  0000 C CNN
+F 2 "LEDs:LED_0805_HandSoldering" V 5725 4000 50  0001 C CNN
 F 3 "" V 5725 4000 50  0000 C CNN
 	1    5725 4000
@@
 F 0 "D1" H 5675 3875 50  0000 L CNN
 F 1 "LED0" H 5800 3700 50  0000 L CNN
-F 2 "" V 5725 3750 50  0000 C CNN
+F 2 "LEDs:LED_0805_HandSoldering" V 5725 3750 50  0001 C CNN
 F 3 "" V 5725 3750 50  0000 C CNN
 	1    5725 3750
@@
 F 0 "D3" H 5675 4425 50  0000 L CNN
 F 1 "LED2" H 5800 4250 50  0000 L CNN
-F 2 "" V 5725 4300 50  0000 C CNN
+F 2 "LEDs:LED_0805_HandSoldering" V 5725 4300 50  0001 C CNN
 F 3 "" V 5725 4300 50  0000 C CNN
 	1    5725 4300
@@
 Wire Wire Line
 	5125 4300 5625 4300
-Connection ~ 5125 4200
 Wire Wire Line
 	5500 4100 5500 4000
 Wire Wire Line
 	5500 4000 5625 4000
-Connection ~ 5025 4100
 Wire Wire Line
 	5350 4000 5350 3750
 Wire Wire Line
 	5350 3750 5625 3750
-Connection ~ 4925 4000
 $Comp
 L R_Small R7
@@
 F 0 "R7" V 6225 3700 50  0000 L CNN
 F 1 "1K" V 6125 3700 50  0000 L CNN
-F 2 "" H 6125 3750 50  0000 C CNN
+F 2 "Resistors_SMD:R_0805_HandSoldering" H 6125 3750 50  0001 C CNN
 F 3 "" H 6125 3750 50  0000 C CNN
 	1    6125 3750
@@
 F 0 "R8" V 6225 3950 50  0000 L CNN
 F 1 "1K" V 6125 3950 50  0000 L CNN
-F 2 "" H 6125 4000 50  0000 C CNN
+F 2 "Resistors_SMD:R_0805_HandSoldering" H 6125 4000 50  0001 C CNN
 F 3 "" H 6125 4000 50  0000 C CNN
 	1    6125 4000
@@
 F 0 "R9" V 6225 4250 50  0000 L CNN
 F 1 "1K" V 6125 4250 50  0000 L CNN
-F 2 "" H 6125 4300 50  0000 C CNN
+F 2 "Resistors_SMD:R_0805_HandSoldering" H 6125 4300 50  0001 C CNN
 F 3 "" H 6125 4300 50  0000 C CNN
 	1    6125 4300
@@
 Text Notes 7750 5325 0    60   ~ 0
 Fast and Low power mode:\n\nLPMB Option features\n\nVDD Fast mode\n\nopen Low Power mode
+Connection ~ 5025 4100
+Wire Wire Line
+	5125 3375 5125 4300
+Wire Wire Line
+	2075 1425 2075 1525
+Wire Wire Line
+	1550 1825 1550 2450
+Connection ~ 1550 2450
+Wire Wire Line
+	1475 1725 1475 3050
+Wire Wire Line
+	1400 1625 1400 3725
+Connection ~ 1400 3725
+Wire Wire Line
+	4925 3175 4925 4000
+Connection ~ 4925 4000
+Wire Wire Line
+	5025 3275 5025 4100
+Connection ~ 5125 4200
 $EndSCHEMATC
